File: blink_555.kicad_pcb (KiCad board)
At the start: 2 copper layers, 0 parts

Commit message: working on pcb
Parts:
- added C1: 10uF, Capacitor_SMD:CP_Elec_5x5.4, F.Cu at (17.0, 27.0)
- added C2: 100nF, Capacitor_SMD:C_0603_1608Metric, F.Cu at (11.0, 12.0)
- added D1: LED, LED_SMD:LED_0805_2012Metric, F.Cu at (43.0, 14.0)
- added J1: PWR, Connector_PinHeader_2.54mm:PinHeader_1x02_P2.54mm_Vertical, F.Cu at (5.00, 17.0)
- added R1: 1k, Resistor_SMD:R_0603_1608Metric, F.Cu at (17.0, 17.0)
- added R2: 47k, Resistor_SMD:R_0603_1608Metric, F.Cu at (17.0, 10.0)
- added R3: 150R, Resistor_SMD:R_0603_1608Metric, F.Cu at (36.0, 14.0)
- added U1: NE555P, Package_DIP:DIP-8_W7.62mm, F.Cu at (25.0, 17.0)
Routing:
- net GND: track 0.00 -> 68.7 mm
- net TIMING: track 0.00 -> 42.0 mm
- net VCC: track 0.00 -> 38.3 mm
- net CV: track 0.00 -> 37.5 mm, vias 0 -> 1
- net DISC: track 0.00 -> 26.6 mm
- net OUTPUT: track 0.00 -> 13.5 mm
- net LED_A: track 0.00 -> 7.96 mm
Other:
- board outline added: 50 x 35 mm
